Commit message: FMB insertion: tactile on Cube collision prims, multi-problem envs, sliver-free FMB collision assets
- tactile_utils._object_mesh also reads UsdGeom.Cube collision prims (URDF <box>): the tight_insertion
  L-peg's collisions are two Cubes, so the tactile sensor raised "no meshes under .../Object" there.
  Screwing taxels are bit-identical to 5f29400 (same states, max diff 0.0).
- TactileSensor: one ray-cast mesh per object asset (envs grouped by _object_asset_index_per_env).
- precise_assembly.multi_problems=[...]: env i gets problem i % K (object, hole and goal viz spawned
  round-robin); problems must share the insertion waypoints (true for fmb_*).
- FMB assets regenerated (FoundationTouch tools/fmb_insertion/make_fmb_insertion_assets.py): one link name
  (fmb_peg) for every shape; sector decompositions with no sliver pieces (the old CDT pieces and 1.8 x 150 mm
  arch-peg pieces failed PhysX GPU cooking and then did not collide at all); arch/star notches filled to
  their convex hull (<= 1.0 / 0.4 mm of material); thin prisms cut to <= 42:1. Every shape now fits its hole
  in a jittered drop test and stays seated.

Co-Authored-By: Claude Opus 5.5 <noreply@anthropic.com>

File: assets/urdf/fmb_insertion/arch/hole_tol0p5mm/fmb_arch_hole_tol0p5mm.urdf (robot description, URDF)
Before this commit: robot fmb_arch_hole_tol0p5mm, 1 links, 0 joints
Links:
- link hole: geometry collision box size=0.08 0.08 0.01; collision mesh filename=hole_coll_000.obj scale=1 1 1

File: assets/urdf/fmb_insertion/arch/peg/fmb_arch_peg.urdf (robot description, URDF)
Before this commit: robot fmb_arch_peg, 1 links, 0 joints
Links:
- removed link fmb_arch_peg
- added link fmb_peg, mass 0.057800; collision mesh filename=peg_coll_00.obj scale=1 1 1; collision mesh filename=peg_coll_01.obj scale=1 1 1

File: assets/urdf/fmb_insertion/circle/peg/fmb_circle_peg.urdf (robot description, URDF)
Before this commit: robot fmb_circle_peg, 1 links, 0 joints
Links:
- removed link fmb_circle_peg
- added link fmb_peg, mass 0.057800; collision mesh filename=peg_coll_00.obj scale=1 1 1; collision mesh filename=peg_coll_01.obj scale=1 1 1

File: assets/urdf/fmb_insertion/ellipse/hole_tol0p5mm/fmb_ellipse_hole_tol0p5mm.urdf (robot description, URDF)
Before this commit: robot fmb_ellipse_hole_tol0p5mm, 1 links, 0 joints
Links:
- link hole: geometry collision box size=0.08 0.08 0.01; collision mesh filename=hole_coll_000.obj scale=1 1 1

File: assets/urdf/fmb_insertion/ellipse/peg/fmb_ellipse_peg.urdf (robot description, URDF)
Before this commit: robot fmb_ellipse_peg, 1 links, 0 joints
Links:
- removed link fmb_ellipse_peg
- added link fmb_peg, mass 0.057800; collision mesh filename=peg_coll_00.obj scale=1 1 1; collision mesh filename=peg_coll_01.obj scale=1 1 1

File: assets/urdf/fmb_insertion/hexagon/hole_tol0p5mm/fmb_hexagon_hole_tol0p5mm.urdf (robot description, URDF)
Before this commit: robot fmb_hexagon_hole_tol0p5mm, 1 links, 0 joints
Links:
- link hole: geometry collision box size=0.08 0.08 0.01; collision mesh filename=hole_coll_000.obj scale=1 1 1

File: assets/urdf/fmb_insertion/hexagon/peg/fmb_hexagon_peg.urdf (robot description, URDF)
Before this commit: robot fmb_hexagon_peg, 1 links, 0 joints
Links:
- removed link fmb_hexagon_peg
- added link fmb_peg, mass 0.057800; collision mesh filename=peg_coll_00.obj scale=1 1 1; visual mesh filename=peg_visual.obj scale=1 1 1

File: assets/urdf/fmb_insertion/rrect/hole_tol0p5mm/fmb_rrect_hole_tol0p5mm.urdf (robot description, URDF)
Before this commit: robot fmb_rrect_hole_tol0p5mm, 1 links, 0 joints
Links:
- link hole: geometry collision box size=0.08 0.08 0.01; collision mesh filename=hole_coll_000.obj scale=1 1 1

File: assets/urdf/fmb_insertion/rrect/peg/fmb_rrect_peg.urdf (robot description, URDF)
Before this commit: robot fmb_rrect_peg, 1 links, 0 joints
Links:
- removed link fmb_rrect_peg
- added link fmb_peg, mass 0.057800; collision mesh filename=peg_coll_00.obj scale=1 1 1; collision mesh filename=peg_coll_01.obj scale=1 1 1

File: assets/urdf/fmb_insertion/star/hole_tol0p5mm/fmb_star_hole_tol0p5mm.urdf (robot description, URDF)
Before this commit: robot fmb_star_hole_tol0p5mm, 1 links, 0 joints
Links:
- link hole: geometry collision box size=0.08 0.08 0.01; collision mesh filename=hole_coll_000.obj scale=1 1 1

File: assets/urdf/fmb_insertion/star/peg/fmb_star_peg.urdf (robot description, URDF)
Before this commit: robot fmb_star_peg, 1 links, 0 joints
Links:
- removed link fmb_star_peg
- added link fmb_peg, mass 0.057800; collision mesh filename=peg_coll_00.obj scale=1 1 1; collision mesh filename=peg_coll_01.obj scale=1 1 1
