Commit message: ContactBench card: one box collision (SDF card was unstable against the SDF holder)
Co-Authored-By: Claude Opus 5.5 <noreply@anthropic.com>

File: assets/urdf/contactbench/objects/card/card.urdf (robot description, URDF)
Before this commit: robot cb_card, 1 links, 0 joints
Links:
- link object: geometry collision box size=0.085000 0.055000 0.001200; visual mesh filename=card.obj scale=1 1 1
