Commit message: ContactBench placing under constraints (hang ruler/wrench, cup stacks n1-3, utensil into vertical bin n0/2), CoACD collision for thin/hollow parts, explicit waypoints; Play env: external object URDFs (assets.object_urdfs / object_scales)
Co-Authored-By: Claude Opus 5.5 <noreply@anthropic.com>

File: assets/urdf/contactbench/objects/allen_key/allen_key.urdf (robot description, URDF)
Before this commit: robot cb_allen_key, 1 links, 0 joints
Links:
- link object: geometry collision mesh filename=coll_00.obj scale=1 1 1; collision mesh filename=coll_01.obj scale=1 1 1

File: assets/urdf/contactbench/objects/cup/cup.urdf (robot description, URDF)
Before this commit: robot cb_cup, 1 links, 0 joints
Links:
- link object: geometry collision mesh filename=coll_00.obj scale=1 1 1; collision mesh filename=coll_01.obj scale=1 1 1

File: assets/urdf/contactbench/objects/key_1/key_1.urdf (robot description, URDF)
Before this commit: robot cb_key_1, 1 links, 0 joints
Links:
- link object: geometry collision mesh filename=coll_00.obj scale=1 1 1; collision mesh filename=coll_01.obj scale=1 1 1

File: assets/urdf/contactbench/objects/spoon/spoon.urdf (robot description, URDF)
Before this commit: robot cb_spoon, 1 links, 0 joints
Links:
- link object: geometry collision mesh filename=coll_00.obj scale=1 1 1; collision mesh filename=coll_01.obj scale=1 1 1

File: assets/urdf/contactbench/objects/wrench/wrench.urdf (robot description, URDF)
Before this commit: robot cb_wrench, 1 links, 0 joints
Links:
- link object: geometry collision mesh filename=coll_00.obj scale=1 1 1; collision mesh filename=coll_01.obj scale=1 1 1
