Commit message: contactbench: cup = exact convex pieces (base + 24 wall sectors), cup stacks collide as exact pieces of the bottom + top fused cup, cb_cuptop_n{2,3,4,6}_lift (lift-only), cup_stack_n4 / cb_cupstack_n4
Co-Authored-By: Claude Opus 5.5 <noreply@anthropic.com>

File: assets/urdf/contactbench/fixtures/cup_stack_n1/cup_stack_n1.urdf (robot description, URDF)
Before this commit: robot cb_cup_stack_n1, 1 links, 0 joints
Links:
- link receptive: geometry collision mesh filename=coll_000.obj scale=1 1 1; collision mesh filename=coll_001.obj scale=1 1 1

File: assets/urdf/contactbench/fixtures/cup_stack_n2/cup_stack_n2.urdf (robot description, URDF)
Before this commit: robot cb_cup_stack_n2, 1 links, 0 joints
Links:
- link receptive: geometry collision mesh filename=coll_000.obj scale=1 1 1; collision mesh filename=coll_001.obj scale=1 1 1

File: assets/urdf/contactbench/fixtures/cup_stack_n3/cup_stack_n3.urdf (robot description, URDF)
Before this commit: robot cb_cup_stack_n3, 1 links, 0 joints
Links:
- link receptive: geometry collision mesh filename=coll_000.obj scale=1 1 1; collision mesh filename=coll_001.obj scale=1 1 1

File: assets/urdf/contactbench/objects/cup/cup.urdf (robot description, URDF)
Before this commit: robot cb_cup, 1 links, 0 joints
Links:
- link object: geometry collision mesh filename=coll_00.obj scale=1 1 1; collision mesh filename=coll_01.obj scale=1 1 1
