Commit message: precise_assembly: object_max_depenetration_velocity (object + distractors; 1000 default launched keychain parts); keychain mat collides as a box instead of an SDF-512
Co-Authored-By: Claude Opus 5.5 <noreply@anthropic.com>

File: assets/urdf/contactbench/fixtures/keychain_mat/keychain_mat.urdf (robot description, URDF)
Before this commit: robot cb_keychain_mat, 1 links, 0 joints
Links:
- link receptive: geometry collision box size=0.12 0.12 0.001; visual mesh filename=keychain_mat.obj scale=1 1 1

Commit message: keychain: restore the settled, threaded cb_keychain_key_1/_key_fob problems and the 160 mm mat from 0158fc7 (4056be1-line metas had the unsettled hanging poses: the bunch dropped 5 cm at reset and the keys came off the ring); object_solver_position_iterations option
Co-Authored-By: Claude Opus 5.5 <noreply@anthropic.com>

File: assets/urdf/contactbench/fixtures/keychain_mat/keychain_mat.urdf (robot description, URDF)
Before this commit: robot cb_keychain_mat, 1 links, 0 joints
Links:
- link receptive: geometry collision box size=0.16 0.16 0.001; visual mesh filename=keychain_mat.obj scale=1 1 1
